File: hardware/kicad/smart-puck.kicad_sch (KiCad schematic)
At the start: 0 parts

Commit message: added some ICs, will need to grab symbols and footprints for the rest of the ICs
Parts:
- added U1: ESP32-C6-MINI-1, RF_Module:ESP32-C6-MINI-1, symbol RF_Module:ESP32-C6-MINI-1
- added U2: TPS63900, Package_SON:WSON-10-1EP_2.5x2.5mm_P0.5mm_EP1.2x2mm_ThermalVias, symbol Regulator_Switching:TPS63900
- added U3: SHT4x, Sensor_Humidity:Sensirion_DFN-4_1.5x1.5mm_P0.8mm_SHT4x_NoCentralPad, symbol Sensor_Humidity:SHT4x
Connections:
- new net: U1.1 (GND), U1.11 (GND), U1.14 (GND), U1.2 (GND), U1.36 (GND), U1.37 (GND), U1.38 (GND), U1.39 (GND), U1.40 (GND), U1.41 (GND), U1.42 (GND), U1.43 (GND), U1.44 (GND), U1.45 (GND), U1.46 (GND), U1.47 (GND), U1.48 (GND), U1.49 (GND), U1.50 (GND), U1.51 (GND), U1.52 (GND), U1.53 (GND)
- new net: U2.11 (GND), U2.8 (GND)

Commit message: worked on schematic
Parts:
- added C1: 22uF 1mOhm, symbol Device:C
- added C2: 10uF 1mOhm, symbol Device:C
- added C3: 1uF, symbol Device:C
- added C4: 10uF, symbol Device:C
- added J1: USB_C_Receptacle_USB2.0_16P, symbol Connector:USB_C_Receptacle_USB2.0_16P
- added J2: HLK-LD2420, Connector_PinSocket_2.54mm:PinSocket_1x05_P2.54mm_Vertical, symbol Connector:Conn_01x05_Socket
- added J3: Battery, symbol Connector_Generic:Conn_01x02
- added L1: 2.2uH 30mOhm, symbol Device:L
- added R1: 36.5kOhm, symbol Device:R
- added R2, R3: 5.1kOhm, symbol Device:R
- added R4: 10kOhm, symbol Device:R
- added U4: BQ25185DLHR, BQ25185:WSON10_DLH_TEX, symbol BQ25185:BQ25185DLHR
- added U5: MAX17048G+T10, MAX17048G:21-0168E_T822-3_MXM, symbol MAX17048G:MAX17048G+T10
Connections:
- net GND: now reaches U1.1 (GND), U1.11 (GND), U1.14 (GND), U1.2 (GND), U1.36 (GND), U1.37 (GND), U1.38 (GND), U1.39 (GND), U1.40 (GND), U1.41 (GND), U1.42 (GND), U1.43 (GND), U1.44 (GND), U1.45 (GND), U1.46 (GND), U1.47 (GND), U1.48 (GND), U1.49 (GND), U1.50 (GND), U1.51 (GND), U1.52 (GND), U1.53 (GND)
- net GND: now also U2.11 (GND), U2.4 (CFG2), U2.5 (CFG3), U2.8 (GND), U3.4 (VSS), C1.1, C2.1, C3.2, C4.1, J1.A1 (GND), J1.A12 (GND), J1.B1 (GND), J1.B12 (GND), J1.SH (SHIELD), J2.2 (Pin_2), R1.1, R2.2, R3.2, R4.2, U4.11 (EPAD), U4.4 (/CE), U4.5 (GND), U5.4 (GND)
- net D-: now reaches U1.17 (IO12)
- net D-: now also J1.A7 (D-), J1.B7 (D-)
- net D+: now reaches U1.18 (IO13)
- net D+: now also J1.A6 (D+), J1.B6 (D+)
- net +3.3V: now reaches U1.3 (3V3)
- net +3.3V: now also U2.6 (VOUT), U3.3 (VDD), C1.2, J2.1 (Pin_1)
- net at U2.1 (EN): now also U2.10 (VIN), U2.2 (SEL), C2.2
- net at U2.3 (CFG1): now also R1.2
- net at U2.7 (LX2): now also L1.1
- net at U2.9 (LX1): now also L1.2
- new net: R4.1, U4.6 (TS/MR)
- new net: J1.A5 (CC1), R2.1
- new net: J1.B5 (CC2), R3.1
- new net: C4.2, U4.1 (SYS)
- new net +5V: J1.A4 (VBUS), J1.A9 (VBUS), J1.B4 (VBUS), J1.B9 (VBUS), U4.10 (IN)
- new net BAT+: C3.1, J3.1 (Pin_1), U4.2 (BAT)
- new net BAT-: J3.2 (Pin_2)
- no-connect marks 0 -> 4
Other:
- note added: "+3.3V GND TX RX OT2"
- moved on the sheet: U1

Commit message: worked on schematic
Parts:
- added C5, C7: 1uF, symbol Device:C
- added C6: 0.1uF, symbol Device:C
- added D1: LED_GKBR, symbol Device:LED_GKBR
- added R10, R9: 68Ohm, symbol Device:R
- added R11: 100Ohm, symbol Device:R
- added R12, R13: 10kOhm, symbol Device:R
- added R5: 18kOhm, symbol Device:R
- added R6: 1kOhm, symbol Device:R
- added R7, R8: 4.7kOhm, symbol Device:R
- added SW1: SW_MEC_5E, symbol Switch:SW_MEC_5E
- C1: value 22uF 1mOhm -> 22uF
- C2: value 10uF 1mOhm -> 10uF
- J1: footprint (none) -> Connector_USB:USB_C_Receptacle_G-Switch_GT-USB-7010ASV
- J3: footprint (none) -> Connector_JST:JST_PH_S2B-PH-K_1x02_P2.00mm_Horizontal
Connections:
- net BAT- is gone; now on net GND: J3.2 (Pin_2)
- net +3.3V: now also R12.2, R13.2, R7.1, R8.1
- net +5V: now also C5.1
- net BAT+: now also C2.2, U2.1 (EN), U2.10 (VIN), U2.2 (SEL), U5.3 (VDD), C6.1
- net GND: now also U5.1 (CTG), U5.6 (QSTRT), U5.9 (EPAD), C5.2, C6.2, C7.2, D1.2 (K), R5.2, R6.2
- net OT2: now reaches U1.12 (IO0)
- net OT2: now also J2.5 (Pin_5)
- net BOOT: now reaches U1.22 (IO8)
- net BOOT: now also SW1.3 (K), SW1.4 (A)
- net RX: now reaches U1.24 (IO18)
- net RX: now also J2.4 (Pin_4)
- net TX: now reaches U1.25 (IO19)
- net TX: now also J2.3 (Pin_3)
- net LED_R: now reaches U1.27 (IO21)
- net LED_R: now also R11.1
- net LED_G: now reaches U1.28 (IO22)
- net LED_G: now also R10.1
- net LED_B: now reaches U1.29 (IO23)
- net LED_B: now also R9.1
- net SDA: now reaches U1.5 (IO2)
- net SDA: now also U3.1 (SDA), U5.8 (SDA), R7.2
- net SCL: now reaches U1.6 (IO3)
- net SCL: now also U3.2 (SCL), U5.7 (SCL), R8.2
- net EN: now reaches U1.8 (EN)
- net EN: now also C7.1, R12.1
- net at U4.7 (ILIM/VSET): now also R5.1
- net at U4.8 (ISET): now also R6.1
- new net: D1.1 (GA), R10.2
- new net: D1.4 (RA), R11.2
- new net: R13.1, SW1.1, SW1.2
- new net: D1.3 (BA), R9.2
- no-connect marks 4 -> 6
Other:
- moved on the sheet: C1, C2, C3, C4, J1, J2, J3, L1, R1, R2, R3, R4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

Commit message: add footprints and start working on pcb layout
Parts:
- C1: footprint (none) -> Capacitor_SMD:C_0603_1608Metric; JLCPCB (none) -> https://jlcpcb.com/partdetail/60514-CL10A226MQ8NRNC/C59461
- C2, C4: footprint (none) -> Capacitor_SMD:C_0603_1608Metric; JLCPCB (none) -> https://jlcpcb.com/partdetail/20411-CL10A106KP8NNNC/C19702
- C3, C5, C7: footprint (none) -> Capacitor_SMD:C_0603_1608Metric; JLCPCB (none) -> https://jlcpcb.com/partdetail/16531-CL10A105KB8NNNC/C15849
- C6: footprint (none) -> Capacitor_SMD:C_0603_1608Metric; JLCPCB (none) -> https://jlcpcb.com/partdetail/YAGEO-CC0603KRX7R9BB104/C14663
- D1: value LED_GKBR -> RS-C1415MBAR; footprint (none) -> RS-C1415MBAR:LED-ARRAY-SMD_4P-L1.6-W1.6-BR-RD-CW
- L1: footprint (none) -> Inductor_SMD:L_TechFuse_SL0624; JLCPCB (none) -> https://jlcpcb.com/partdetail/TECHFUSE-SL06242R2M/C22463811
- R1: footprint (none) -> Resistor_SMD:R_0402_1005Metric; JLCPCB (none) -> https://jlcpcb.com/partdetail/Walsin_TechCorp-WR04X3652FTL/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
- R10, R9: footprint (none) -> Resistor_SMD:R_0402_1005Metric; JLCPCB (none) -> https://jlcpcb.com/partdetail/VO-SCR0402F68R/C3015752
- R11: footprint (none) -> Resistor_SMD:R_0402_1005Metric; JLCPCB (none) -> https://jlcpcb.com/partdetail/25819-0402WGF1000TCE/C25076
- R12, R13, R4: footprint (none) -> Resistor_SMD:R_0805_2012Metric; JLCPCB (none) -> https://jlcpcb.com/partdetail/18102-0805W8F1002T5E/C17414
- R2, R3: footprint (none) -> Resistor_SMD:R_0402_1005Metric; JLCPCB (none) -> https://jlcpcb.com/partdetail/26648-0402WGF5101TCE/C25905
- R5: footprint (none) -> Resistor_SMD:R_0603_1608Metric; JLCPCB (none) -> https://jlcpcb.com/partdetail/26553-0603WAF1802T5E/C25810
- R6: footprint (none) -> Resistor_SMD:R_0603_1608Metric; JLCPCB (none) -> https://jlcpcb.com/partdetail/21904-0603WAF1001T5E/C21190
- R7, R8: footprint (none) -> Resistor_SMD:R_0402_1005Metric; JLCPCB (none) -> https://jlcpcb.com/partdetail/26643-0402WGF4701TCE/C25900
- SW1: value SW_MEC_5E -> GT-TZ084B-H015-L1; footprint (none) -> GT-TZ084B-H015-L1:SW-SMD_4P-L5.2-W5.2-P3.70-LS6.4
